File: Test Hardware/Training Loadboard/Training_LB/Training_LB.kicad_sch (KiCad schematic)
At the start: 18 parts, among them J1 DUT64, J2 DUT64, J3 DUT64, J4 DUT64, J5 DUT64, J6 DUT64, J7 DUT64, J8 DUT64, U1 MCP3008, U2 MCP4901

Commit message: EOD Office
Parts:
- added C10, C12, C14, C16, C18, C20, C22, C24, C26, C28, C30, C32, C34, C36, C38, C40, C42, C44, C46, C48: 10uF, Capacitor_SMD:C_1206_3216Metric_Pad1.33x1.80mm_HandSolder, symbol Device:C_Small
- added C11, C13, C15, C17, C19, C21, C23, C25, C27, C29, C31, C33, C35, C37, C39, C41, C43, C45, C47, C9: 0.1uF, Capacitor_SMD:C_1206_3216Metric_Pad1.33x1.80mm_HandSolder, symbol Device:C_Small
- added U10, U14, U15, U16: NE555D, Package_SO:SOIC-8_3.9x4.9mm_P1.27mm, symbol Timer:NE555D
- added U11, U12, U13, U9: 74HC595, symbol 74xx:74HC595
- added U3, U4, U5: MCP3008, Training_Lib:SOIC16-N_MC_MCH, symbol Analog_ADC:MCP3008
- added U6, U7, U8: MCP4901, symbol Analog_DAC:MCP4901
Connections:
- net GND: now also C10.2, C11.2, C12.2, C13.2, C14.2, C15.2, C16.2, C17.2, C18.2, C19.2, C20.2, C21.2, C22.2, C23.2, C24.2, C25.2, C26.2, C27.2, C28.2, C29.2, C30.2, C31.2, C32.2, C33.2, C34.2, C35.2, C36.2, C37.2, C38.2, C39.2, C40.2, C41.2, C42.2, C43.2, C44.2, C45.2, C46.2, C47.2, C48.2, C9.2, U10.1 (GND), U11.8 (GND), U12.8 (GND), U13.8 (GND), U14.1 (GND), U15.1 (GND), U16.1 (GND), U3.14 (AGND), U3.9 (DGND), U4.14 (AGND), U4.9 (DGND), U5.14 (AGND), U5.9 (DGND), U9.8 (GND)
- net Vss: now also U6.15 (Vss), U7.15 (Vss), U8.15 (Vss)
- net 225P16: now reaches J1.1
- net 330PS1: now reaches J1.10
- net 330GS1: now reaches J1.11
- net D10306: now reaches J1.12
- net D10304: now reaches J1.13
- net D10301: now reaches J1.14
- net D10305: now reaches J1.15
- net URW01_2: now reaches J1.16
- net 425P16: now reaches J1.17
- net 425PS16: now reaches J1.18
- net 431_MESE_D-: now reaches J1.19
- net 225PS16: now reaches J1.2
- net 431_MESE_D+: now reaches J1.20
- net UP5V: now reaches J1.21
- net D0213: now reaches J1.22
- net D10303: now reaches J1.23
- net D10302: now reaches J1.24
- net 330P3: now reaches J1.25
- net 330PS3: now reaches J1.26
- net 330GS3: now reaches J1.27
- net D10212: now reaches J1.28
- net D10210: now reaches J1.29
- net D10311: now reaches J1.3
- net D10208: now reaches J1.30
- net D10211: now reaches J1.31
- net D10209: now reaches J1.32
- net D10310: now reaches J1.4
- net URW00_2: now reaches J1.5
- net D10308: now reaches J1.6
- net D10309: now reaches J1.7
- net D10307: now reaches J1.8
- net 330P1: now reaches J1.9
- net 329-GS3: now reaches J2.1
- net D10105: now reaches J2.10
- net 225-PS14: now reaches J2.11
- net 225-P14: now reaches J2.12
- net D10110: now reaches J2.13
- net 329-P3: now reaches J2.14
- net D10113: now reaches J2.15
- net 425-P14: now reaches J2.16
- net D10101: now reaches J2.17
- net UW10_2: now reaches J2.18
- net 231-SRCE-H+: now reaches J2.19
- net D10203: now reaches J2.2
- net D10202: now reaches J2.20
- net D10104: now reaches J2.21
- net 329-PS1: now reaches J2.22
- net D10107: now reaches J2.23
- net 231-SRCE-H-: now reaches J2.24
- net D10204: now reaches J2.25
- net 329-GS1: now reaches J2.26
- net UW11_2: now reaches J2.27
- net D10201: now reaches J2.28
- net 329-P1: now reaches J2.29
- net D10109: now reaches J2.3
- net D10111: now reaches J2.30
- net D10206: now reaches J2.31
- net D10106: now reaches J2.32
- net D10108: now reaches J2.4
- net 329-PS3: now reaches J2.5
- net D10207: now reaches J2.6
- net 425-PS14: now reaches J2.7
- net D10112: now reaches J2.8
- net D10205: now reaches J2.9
- net CH2_1: now reaches U1.5 (CH4)
- net CH0 renamed CH0_1
- net CH1: no longer names the net of U1.2 (CH1)
- net CH2 renamed CH1_1
- net CH3: no longer names the net of U1.4 (CH3)
- net CLK_MCP3008 renamed CLK_MCP3008_1
- net CS_MCP3008 renamed CS_MCP3008_1
- net CS_MCP4901 renamed CS_MCP4901_1
- net Din renamed Din_1
- net Dout renamed Dout_1
- net LDAC renamed LDAC_1
- net SCK renamed SCK_1
- net SDI renamed SDI_1
- net Vdd_MCP3008 renamed Vdd_MCP3008_1
- net Vdd_MCP4901 renamed Vdd_MCP4901_1
- net Vout renamed Vout_1
- net Vref_MCP3008 renamed Vref_MCP3008_1
- net Vref_MCP4901 renamed Vref_MCP4901_1
- new net CH0_2: U3.1 (CH0)
- new net CH0_3: U4.1 (CH0)
- new net CH0_4: U5.1 (CH0)
- new net CH1_2: U3.3 (CH2)
- new net CH1_3: U4.3 (CH2)
- new net CH1_4: U5.3 (CH2)
- new net CH2_2: U3.5 (CH4)
- new net CH2_3: U4.5 (CH4)
- new net CH2_4: U5.5 (CH4)
- new net CLK_MCP3008_2: U3.13 (CLK)
- new net CLK_MCP3008_3: U4.13 (CLK)
- new net CLK_MCP3008_4: U5.13 (CLK)
- new net CONT_1: U10.5 (CONT)
- new net CONT_2: U14.5 (CONT)
- new net CONT_3: U15.5 (CONT)
- new net CONT_4: U16.5 (CONT)
- new net CS_MCP3008_2: U3.10 (~{CS}/SHDN)
- new net CS_MCP3008_3: U4.10 (~{CS}/SHDN)
- new net CS_MCP3008_4: U5.10 (~{CS}/SHDN)
- new net CS_MCP4901_2: U8.2 (~{CS})
- new net CS_MCP4901_3: U6.2 (~{CS})
- new net CS_MCP4901_4: U7.2 (~{CS})
- new net DISCH_1: U10.7 (DISCH)
- new net DISCH_2: U14.7 (DISCH)
- new net DISCH_3: U15.7 (DISCH)
- new net DISCH_4: U16.7 (DISCH)
- new net Din_2: U3.11 (Din)
- new net Din_3: U4.11 (Din)
- new net Din_4: U5.11 (Din)
- new net Dout_2: U3.12 (Dout)
- new net Dout_3: U4.12 (Dout)
- new net Dout_4: U5.12 (Dout)
- new net LDAC_2: U8.13 (~{LDAC})
- new net LDAC_3: U6.13 (~{LDAC})
- new net LDAC_4: U7.13 (~{LDAC})
- new net OUT_1: U10.3 (OUT)
- new net OUT_2: U14.3 (OUT)
- new net OUT_3: U15.3 (OUT)
- new net OUT_4: U16.3 (OUT)
- new net Q0_1: U9.15 (QA)
- new net Q0_2: U11.15 (QA)
- new net Q0_3: U12.15 (QA)
- new net Q0_4: U13.15 (QA)
- new net Q1_1: U9.1 (QB)
- new net Q1_2: U11.1 (QB)
- new net Q1_3: U12.1 (QB)
- new net Q1_4: U13.1 (QB)
- new net Q2_1: U9.2 (QC)
- new net Q2_2: U11.2 (QC)
- new net Q2_3: U12.2 (QC)
- new net Q2_4: U13.2 (QC)
- new net Q3_1: U9.3 (QD)
- new net Q3_2: U11.3 (QD)
- new net Q3_3: U12.3 (QD)
- new net Q3_4: U13.3 (QD)
- new net Q4_1: U9.4 (QE)
- new net Q4_2: U11.4 (QE)
- new net Q4_3: U12.4 (QE)
- new net Q4_4: U13.4 (QE)
- new net Q5_1: U9.5 (QF)
- new net Q5_2: U11.5 (QF)
- new net Q5_3: U12.5 (QF)
- new net Q5_4: U13.5 (QF)
- new net Q6_1: U9.6 (QG)
- new net Q6_2: U11.6 (QG)
- new net Q6_3: U12.6 (QG)
- new net Q6_4: U13.6 (QG)
- new net Q7_1: U9.7 (QH)
- new net Q7_2: U11.7 (QH)
- new net Q7_3: U12.7 (QH)
- new net Q7_4: U13.7 (QH)
- new net RCLK_1: U9.12 (RCLK)
- new net RCLK_2: U11.12 (RCLK)
- new net RCLK_3: U12.12 (RCLK)
- new net RCLK_4: U13.12 (RCLK)
- new net SCK_2: U8.3 (SCK)
- new net SCK_3: U6.3 (SCK)
- new net SCK_4: U7.3 (SCK)
- new net SDI_2: U8.4 (SDI)
- new net SDI_3: U6.4 (SDI)
- new net SDI_4: U7.4 (SDI)
- new net SER_1: U9.14 (SER)
- new net SER_2: U11.14 (SER)
- new net SER_3: U12.14 (SER)
- new net SER_4: U13.14 (SER)
- new net SRCLK_1: U9.11 (SRCLK)
- new net SRCLK_2: U11.11 (SRCLK)
- new net SRCLK_3: U12.11 (SRCLK)
- new net SRCLK_4: U13.11 (SRCLK)
- new net THRES_1: U10.6 (THRES)
- new net THRES_2: U14.6 (THRES)
- new net THRES_3: U15.6 (THRES)
- new net THRES_4: U16.6 (THRES)
- new net TRIG_1: U10.2 (TRIG)
- new net TRIG_2: U14.2 (TRIG)
- new net TRIG_3: U15.2 (TRIG)
- new net TRIG_4: U16.2 (TRIG)
- new net VCC_74HC595_1: C33.1, C34.1, U9.10 (~{SRCLR}), U9.16 (VCC)
- new net VCC_74HC595_2: C35.1, C36.1, U11.10 (~{SRCLR}), U11.16 (VCC)
- new net VCC_74HC595_3: C37.1, C38.1, U12.10 (~{SRCLR}), U12.16 (VCC)
- new net VCC_74HC595_4: C39.1, C40.1, U13.10 (~{SRCLR}), U13.16 (VCC)
- new net VCC_NE555_1: C41.1, C42.1, U10.8 (VCC)
- new net VCC_NE555_2: C43.1, C44.1, U14.8 (VCC)
- new net VCC_NE555_3: C45.1, C46.1, U15.8 (VCC)
- new net VCC_NE555_4: C47.1, C48.1, U16.8 (VCC)
- new net Vdd_MCP3008_2: C10.1, C9.1, U3.16 (Vdd)
- new net Vdd_MCP3008_3: C13.1, C14.1, U4.16 (Vdd)
- new net Vdd_MCP3008_4: C17.1, C18.1, U5.16 (Vdd)
- new net Vdd_MCP4901_2: C29.1, C30.1, U8.1 (Vdd)
- new net Vdd_MCP4901_3: C21.1, C22.1, U6.1 (Vdd)
- new net Vdd_MCP4901_4: C25.1, C26.1, U7.1 (Vdd)
- new net Vout_2: U8.16 (Vout)
- new net Vout_3: U6.16 (Vout)
- new net Vout_4: U7.16 (Vout)
- new net Vref_MCP3008_2: C11.1, C12.1, U3.15 (Vref)
- new net Vref_MCP3008_3: C15.1, C16.1, U4.15 (Vref)
- new net Vref_MCP3008_4: C19.1, C20.1, U5.15 (Vref)
- new net Vref_MCP4901_2: C31.1, C32.1, U8.14 (Vref)
- new net Vref_MCP4901_3: C23.1, C24.1, U6.14 (Vref)
- new net Vref_MCP4901_4: C27.1, C28.1, U7.14 (Vref)
- new net _OE_1: U9.13 (~{OE})
- new net _OE_2: U11.13 (~{OE})
- new net _OE_3: U12.13 (~{OE})
- new net _OE_4: U13.13 (~{OE})
- new net _Q7_1: U9.9 (QH')
- new net _Q7_2: U11.9 (QH')
- new net _Q7_3: U12.9 (QH')
- new net _Q7_4: U13.9 (QH')
- new net _RST_1: U10.4 (~{RST})
- new net _RST_2: U14.4 (~{RST})
- new net _RST_3: U15.4 (~{RST})
- new net _RST_4: U16.4 (~{RST})
- no-connect marks 268 -> 244
Other:
- moved on the sheet: C1, C2, C3, C4, C5, C6, C7, C8, J1, J2, J3, J4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

Commit message: EOD Office
Connections:
- net 225-P14: now also J4.12, J5.21, J7.21
- net 225-PS14: now also J4.11, J5.22, J7.22
- net 225P16: now also J3.1, J6.32, J8.32
- net 225PS16: now also J3.2, J6.31, J8.31
- net 231-SRCE-H+: now also J4.19, J5.14, J7.14
- net 231-SRCE-H-: now also J4.24, J5.9, J7.9
- net 329-GS1: now also J4.26, J5.7, J7.7
- net 329-GS3: now also J4.1, J5.32, J7.32
- net 329-P1: now also J4.29, J5.4, J7.4
- net 329-P3: now also J4.14, J5.19, J7.19
- net 329-PS1: now also J4.22, J5.11, J7.11
- net 329-PS3: now also J4.5, J5.28, J7.28
- net 330GS1: now also J3.11, J6.22, J8.22
- net 330GS3: now also J3.27, J6.6, J8.6
- net 330P1: now also J3.9, J6.24, J8.24
- net 330P3: now also J3.25, J6.8, J8.8
- net 330PS1: now also J3.10, J6.23, J8.23
- net 330PS3: now also J3.26, J6.7, J8.7
- net 425-P14: now also J4.16, J5.17, J7.17
- net 425-PS14: now also J4.7, J5.26, J7.26
- net 425P16: now also J3.17, J6.16, J8.16
- net 425PS16: now also J3.18, J6.15, J8.15
- net 431_MESE_D+: now also J3.20, J6.13, J8.13
- net 431_MESE_D-: now also J3.19, J6.14, J8.14
- net D0213: now also J3.22, J6.11, J8.11
- net D10101: now also J4.17, J5.16, J7.16
- net D10104: now also J4.21, J5.12, J7.12
- net D10105: now also J4.10, J5.23, J7.23
- net D10106: now also J4.32, J5.1, J7.1
- net D10107: now also J4.23, J5.10, J7.10
- net D10108: now also J4.4, J5.29, J7.29
- net D10109: now also J4.3, J5.30, J7.30
- net D10110: now also J4.13, J5.20, J7.20
- net D10111: now also J4.30, J5.3, J7.3
- net D10112: now also J4.8, J5.25, J7.25
- net D10113: now also J4.15, J5.18, J7.18
- net D10201: now also J4.28, J5.5, J7.5
- net D10202: now also J4.20, J5.13, J7.13
- net D10203: now also J4.2, J5.31, J7.31
- net D10204: now also J4.25, J5.8, J7.8
- net D10205: now also J4.9, J5.24, J7.24
- net D10206: now also J4.31, J5.2, J7.2
- net D10207: now also J4.6, J5.27, J7.27
- net D10208: now also J3.30, J6.3, J8.3
- net D10209: now also J3.32, J6.1, J8.1
- net D10210: now also J3.29, J6.4, J8.4
- net D10211: now also J3.31, J6.2, J8.2
- net D10212: now also J3.28, J6.5, J8.5
- net D10301: now also J3.14, J6.19, J8.19
- net D10302: now also J3.24, J6.9, J8.9
- net D10303: now also J3.23, J6.10, J8.10
- net D10304: now also J3.13, J6.20, J8.20
- net D10305: now also J3.15, J6.18, J8.18
- net D10306: now also J3.12, J6.21, J8.21
- net D10307: now also J3.8, J6.25, J8.25
- net D10308: now also J3.6, J6.27, J8.27
- net D10309: now also J3.7, J6.26, J8.26
- net D10310: now also J3.4, J6.29, J8.29
- net D10311: now also J3.3, J6.30, J8.30
- net UP5V: now also J3.21, J6.12, J8.12
- net URW00_2: now also J3.5, J6.28, J8.28
- net URW01_2: now also J3.16, J6.17, J8.17
- net UW10_2: now also J4.18, J5.15, J7.15
- net UW11_2: now also J4.27, J5.6, J7.6
- no-connect marks 244 -> 52
Other:
- moved on the sheet: J3, J4, J5, J6, J7, J8
